File: 30MHz preamp with lna and ant_sw.kicad_pcb (KiCad board)
At the start: 2 copper layers, 32 x 21.2 mm, 17 parts, among them SW1 SW-AMP_ON-OFF, U1 AS179-92LF, U2 BGA2869, U3 MCP1703Ax-500xxMB

Commit message: Add files via upload
Other:
- board size 32 x 21.2 mm -> 33.5 x 21.2 mm
Changed lines of the file:
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@@
 	)
 	(gr_line
-		(start 115.75 87.75)
-		(end 115.75 66.5)
+		(start 148.5 66.5)
+		(end 148.5 87.75)
 		(stroke
 			(width 0.05)
@@
 	)
 	(gr_line
-		(start 147.75 66.5)
-		(end 147.75 87.75)
+		(start 148.5 87.75)
+		(end 115 87.75)
 		(stroke
 			(width 0.05)
@@
 	)
 	(gr_line
-		(start 147.75 87.75)
-		(end 115.75 87.75)
+		(start 115 87.75)
+		(end 115 66.5)
 		(stroke
 			(width 0.05)
@@
 	)
 	(gr_line
-		(start 115.75 66.5)
-		(end 147.75 66.5)
+		(start 115 66.5)
+		(end 148.5 66.5)
 		(stroke
 			(width 0.05)
@@
 		(start 130.25 70.05)
 		(end 130.25 69.4)
-		(width 0.25)
+		(width 0.35)
 		(layer "F.Cu")
 		(net 1)
@@
 		(start 136 71.65)
 		(end 137.35 71.65)
-		(width 0.25)
+		(width 0.35)
 		(layer "F.Cu")
 		(net 1)
@@
 		(start 128.35 69.4)
 		(end 130.25 69.4)
-		(width 0.25)
+		(width 0.35)
 		(layer "F.Cu")
 		(net 1)
@@
 		(start 128.08 79.8)
 		(end 128.08 83.75)
-		(width 0.4)
+		(width 0.45)
 		(layer "F.Cu")
 		(net 2)
@@
 		(start 130.08 79.35)
 		(end 128.53 79.35)
-		(width 0.4)
+		(width 0.45)
 		(layer "F.Cu")
 		(net 2)
@@
 		(start 128.53 79.35)
 		(end 128.08 79.8)
-		(width 0.4)
+		(width 0.45)
 		(layer "F.Cu")
 		(net 2)
@@
 		(start 127.25 67.5)
 		(end 127.25 68.75)
-		(width 0.3)
+		(width 0.4)
 		(layer "F.Cu")
 		(net 2)
@@
 		(start 130.08 79.35)
 		(end 131.29 79.35)
-		(width 0.4)
+		(width 0.45)
 		(layer "F.Cu")
 		(net 2)
@@
 		(start 127.25 68.75)
 		(end 128.35 68.75)
-		(width 0.25)
+		(width 0.35)
 		(layer "F.Cu")
 		(net 2)
@@
 		(start 126.2 68.75)
 		(end 127.25 68.75)
-		(width 0.3)
+		(width 0.4)
 		(layer "F.Cu")
 		(net 2)
@@
 		(start 131.29 79.35)
 		(end 132.79 77.85)
-		(width 0.4)
+		(width 0.45)
 		(layer "F.Cu")
 		(net 2)
@@
 		(start 119.75 70)
 		(end 122.25 67.5)
-		(width 0.4)
+		(width 0.45)
 		(layer "B.Cu")
 		(net 2)
@@
 		(start 128.08 83.75)
 		(end 121.75 83.75)
-		(width 0.4)
+		(width 0.45)
 		(layer "B.Cu")
 		(net 2)
@@
 		(start 121.75 83.75)
 		(end 119.75 81.75)
-		(width 0.4)
+		(width 0.45)
 		(layer "B.Cu")
 		(net 2)
@@
 		(start 119.75 81.75)
 		(end 119.75 70)
-		(width 0.4)
+		(width 0.45)
 		(layer "B.Cu")
 		(net 2)
@@
 		(start 122.25 67.5)
 		(end 127.25 67.5)
-		(width 0.4)
+		(width 0.45)
 		(layer "B.Cu")
 		(net 2)
@@
 		(start 134.25 86.25)
 		(end 134.25 77.9775)
-		(width 0.4)
+		(width 0.45)
 		(layer "F.Cu")
 		(net 3)
@@
 		(start 138.58 79.35)
 		(end 136.7 79.35)
-		(width 0.4)
+		(width 0.45)
 		(layer "F.Cu")
 		(net 3)
@@
 		(start 136.7 79.35)
 		(end 134.25 81.8)
-		(width 0.4)
+		(width 0.45)
 		(layer "F.Cu")
 		(net 3)
@@
 		(start 122.025 72.475)
 		(end 121.25 71.7)
-		(width 0.25)
+		(width 0.4)
 		(layer "F.Cu")
 		(net 4)
@@
 		(start 132.975 71.65)
 		(end 134.1 71.65)
-		(width 0.25)
+		(width 0.35)
 		(layer "F.Cu")
 		(net 4)
@@
 		(start 129.118629 73.25)
 		(end 123.896015 73.25)
-		(width 0.25)
+		(width 0.4)
 		(layer "F.Cu")
 		(net 4)
@@
 		(mid 130.163879 73.042086)
 		(end 129.118629 73.25)
-		(width 0.25)
+		(width 0.4)
 		(layer "F.Cu")
 		(net 4)
@@
 		(mid 122.883429 73.048584)
 		(end 123.896015 73.25)
-		(width 0.25)
+		(width 0.4)
 		(layer "F.Cu")
 		(net 4)
@@
 		(mid 131.935635 71.856742)
 		(end 131.054504 72.445495)
-		(width 0.25)
+		(width 0.4)
 		(layer "F.Cu")
 		(net 4)
@@
 		(start 121.25 69.8)
 		(end 117.41 69.8)
-		(width 0.25)
+		(width 0.45)
 		(layer "F.Cu")
 		(net 5)
@@
 		(start 136 72.3)
 		(end 139.75 72.3)
-		(width 0.25)
+		(width 0.35)
 		(layer "F.Cu")
 		(net 6)
@@
 		(start 141.7 72.25)
 		(end 141.7 68.75)
-		(width 0.25)
+		(width 0.4)
 		(layer "F.Cu")
 		(net 7)
@@
 		(start 143.407106 69.75)
 		(end 146.25 69.75)
-		(width 0.25)
+		(width 0.4)
 		(layer "F.Cu")
 		(net 7)
@@
 		(start 142.2 69.25)
 		(end 141.7 68.75)
-		(width 0.25)
+		(width 0.35)
 		(layer "F.Cu")
 		(net 7)
@@
 		(mid 142.753825 69.620054)
 		(end 143.407106 69.75)
-		(width 0.25)
+		(width 0.4)
 		(layer "F.Cu")
 		(net 7)
@@
 		(start 135.35 71.4)
 		(end 135.75 71)
-		(width 0.25)
+		(width 0.35)
 		(layer "F.Cu")
 		(net 8)
@@
 		(start 136 71)
 		(end 135.75 71)
-		(width 0.2)
+		(width 0.35)
 		(layer "F.Cu")
 		(net 8)
@@
 		(start 134.95 72.365685)
 		(end 134.95 74.5)
-		(width 0.25)
+		(width 0.4)
 		(layer "F.Cu")
 		(net 8)
@@
 		(mid 135.053956 71.84306)
 		(end 134.95 72.365685)
-		(width 0.25)
+		(width 0.4)
 		(layer "F.Cu")
 		(net 8)
@@
 		(start 128.25 74.15)
 		(end 132.7 74.15)
-		(width 0.25)
+		(width 0.4)
 		(layer "F.Cu")
 		(net 9)
@@
 		(start 130.25 68.75)
 		(end 139.8 68.75)
-		(width 0.25)
+		(width 0.35)
 		(layer "F.Cu")
 		(net 10)
@@
 		(start 128.25 72.25)
 		(end 128.25 70.15)
-		(width 0.25)
+		(width 0.4)
 		(layer "F.Cu")
 		(net 11)
@@
 		(start 133.85 70.75)
 		(end 134.1 71)
-		(width 0.2)
+		(width 0.25)
 		(layer "F.Cu")
 		(net 13)
@@
 		(start 132.75 70.75)
 		(end 133.85 70.75)
-		(width 0.2)
+		(width 0.25)
 		(layer "F.Cu")
 		(net 13)
@@
 		(start 133.9 72.5)
 		(end 134.1 72.3)
-		(width 0.2)
+		(width 0.25)
 		(layer "F.Cu")
 		(net 14)
@@
 		(start 132.75 72.5)
 		(end 133.9 72.5)
-		(width 0.2)
+		(width 0.25)
 		(layer "F.Cu")
 		(net 14)
@@
 		(polygon
 			(pts
-				(xy 115.5 66.5) (xy 148 66.5) (xy 148 88) (xy 115.5 88) (xy 115.5 87.75)
+				(xy 115 66.5) (xy 148.5 66.5) (xy 148.5 88) (xy 115 88) (xy 115 87.5)
 			)
 		)

Commit message: Add files via upload
Parts:
- TP3: value +12V -> 8-15V
Changed lines of the file:
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@@
 			)
 		)
-		(property "Value" "+12V"
-			(at 9 0.25 0)
+		(property "Value" "8-15V"
+			(at 9.5 0.25 0)
 			(layer "F.SilkS")
 			(effects
@@
 	)
 	(via
-		(at 123 75.75)
+		(at 123 76)
 		(size 0.6)
 		(drill 0.3)
@@
 	)
 	(via
-		(at 125 75.75)
-		(size 0.6)
-		(drill 0.3)
+		(at 125 76)
+		(size 0.6)
+		(drill 0.3)
