File: 30MHz preamp with lna and ant_sw.kicad_sch (KiCad schematic)
At the start: 17 parts, among them SW1 SW-AMP_ON-OFF, U1 AS179-92LF, U2 BGA2869, U3 MCP1703Ax-500xxMB

Commit message: Add files via upload
Other:
- note added: "Input voltage: 8-15V"
Changed lines of the file:
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@@
 		(company "Z32IT")
+	)
+	(text "Input voltage: 8-15V"
+		(exclude_from_sim no)
+		(at 160.02 91.694 0)
+		(effects
+			(font
+				(size 1 1)
+			)
+		)
 	)
 	(text "-J1-\nV1=J2\nV2=J3"
